File: Hardware/DF45_module.sch (KiCad schematic (older format))
At the start: 85 parts, among them J1 M02PTH, Q1 CSD18537NQ5A, Q2 CSD18537NQ5A, Q3 CSD18537NQ5A, Q4 CSD18537NQ5A, Q5 CSD18537NQ5A, Q6 CSD18537NQ5A, U2 HIP408624-SOIC, U3 74HC153TSSOP-16, U4 74HC153TSSOP-16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

Commit message: Updated hardware to use latest library references.
Parts:
- C1, C10, C11, C12, C13, C14, C15, C16, C17, C18, C19, C2, C20, C21, C22, C3, C4, C6, C7, C8, C9: footprint ee448_driver8:0805-CAP -> Capacitor_SMD:C_0805_2012Metric
- C23: footprint ee448_driver8:PCAP_125X25 -> Capacitor_THT:C_Radial_D12.5mm_H25.0mm_P5.00mm
- CR1, CR2, CR3, CR4, CR5, CR6: footprint ee448_driver8:SD2114 -> Package_SON:VSONP-8-1EP_5x6_P1.27mm
- CSENSE1: footprint ee448_driver8:SO08 -> Package_SO:SOIC-8_3.9x4.9mm_P1.27mm
- D1, D10, D2, D3, D4, D6: footprint ee448_driver8:SMA-DIODE -> Diode_SMD:D_SMA
- D7: footprint ee448_driver8:SMC -> Diode_SMD:D_SMC
- L1, PWR1: footprint ee448_driver8:CHIPLED_0805 -> LED_SMD:LED_0805_2012Metric
- Q1, Q2, Q3, Q4, Q5, Q6: footprint ee448_driver8:DQJ8 -> Package_SON:VSONP-8-1EP_5x6_P1.27mm
- R1, R10, R11, R12, R13, R14, R15, R16, R17, R18, R19, R2, R20, R3, R4, R5, R6, R7, R8, R9: footprint ee448_driver8:0805 -> Resistor_SMD:R_0805_2012Metric
- U2: footprint ee448_driver8:24-SOIC -> Package_SO:SOIC-24W_7.5x15.4mm_P1.27mm
- U3, U4, U5: footprint ee448_driver8:TSSOP-16 -> Package_SO:TSSOP-16_4.4x5mm_P0.65mm
- U6: footprint ee448_driver8:SC70-5 -> Package_TO_SOT_SMD:SOT-353_SC-70-5
- U7: footprint ee448_driver8:32A -> Package_QFP:TQFP-32_7x7mm_P0.8mm
- XTAL1: footprint ee448_driver8:CTS406 -> Crystal:Crystal_SMD_0603-4Pin_6.0x3.5mm
